File: 2013_spring/pb171/RotDisplay.X/schematics/RotDisplay.sch (KiCad schematic (older format))
At the start: 34 parts

Commit message: schema is done
Parts:
- removed R?: R, symbol R
- added R?: 10k, ~, symbol R
- R?: value R -> 180
Connections:
- net labels added: CLK, DAT, N.C., Vdd, Vpp
- wire segments 111 -> 131
- no-connect marks 17 -> 16
Other:
- moved on the sheet: D?, R?
