File: 2013_spring/pb171/RotaryDisplay/schematics/RotDisplay.sch (KiCad schematic (older format))
At the start: 34 parts

Commit message: schema svg
Parts:
- SW?: value SW_PUSH -> PUSH_LEFT
- SW?: value SW_PUSH -> PUSH_RIGHT
- renumbered SW_MCU to MCU_ON, SW_RTC to RTC_ON
Changed lines of the file:
@@
 $EndComp
 $Comp
-L SPST SW_RTC
+L SPST RTC_ON
 U 1 1 51B793EE
 P 8350 1800
-F 0 "SW_RTC" H 8350 1900 70  0000 C CNN
+F 0 "RTC_ON" H 8350 1900 70  0000 C CNN
 F 1 "SPST" H 8350 1700 70  0000 C CNN
 F 2 "" H 8350 1800 60  0001 C CNN
@@
 $EndComp
 $Comp
-L SPST SW_MCU
+L SPST MCU_ON
 U 1 1 51B793D8
 P 7950 1800
-F 0 "SW_MCU" H 7950 1900 70  0000 C CNN
+F 0 "MCU_ON" H 7950 1900 70  0000 C CNN
 F 1 "SPST" H 7950 1700 70  0000 C CNN
 F 2 "" H 7950 1800 60  0001 C CNN
@@
 P 7300 5850
 F 0 "SW?" H 7450 5960 50  0000 C CNN
-F 1 "SW_PUSH" H 7300 5770 50  0000 C CNN
+F 1 "PUSH_RIGHT" H 7300 5770 50  0000 C CNN
 F 2 "" H 7300 5850 60  0001 C CNN
 F 3 "" H 7300 5850 60  0001 C CNN
@@
 P 6800 5850
 F 0 "SW?" H 6950 5960 50  0000 C CNN
-F 1 "SW_PUSH" H 6800 5770 50  0000 C CNN
+F 1 "PUSH_LEFT" H 6800 5770 50  0000 C CNN
 F 2 "" H 6800 5850 60  0001 C CNN
 F 3 "" H 6800 5850 60  0001 C CNN
